File: untitled.kicad_sch (KiCad schematic)
At the start: 154 parts, among them J1 Conn_02x05_Odd_Even, J2 Conn_02x05_Odd_Even, J3 Conn_02x05_Odd_Even, J5 Conn_02x05_Odd_Even, J6 Conn_02x05_Odd_Even, SW1 KAD08LHGT, SW10 KAD08LHGT, SW11 SW_Push, SW12 SW_Push, SW13 SW_Push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

Commit message: Finalized PORTS
Connections:
- net VCC_MCU renamed +3.3V
